File: DIY_Keyboard.kicad_pcb (KiCad board)
At the start: 2 copper layers, 357.7 x 136.8 mm, 170 parts, among them SW1 SW_Push, SW10 SW_Push, SW11 SW_Push, SW12 SW_Push, SW13 SW_Push, SW14 SW_Push, SW15 SW_Push, SW16 SW_Push, SW17 SW_Push, SW18 SW_Push, SW19 SW_Push, SW2 SW_Push, SW20 SW_Push, SW21 SW_Push, SW22 SW_Push, SW23 SW_Push, SW24 SW_Push, SW25 SW_Push, SW26 SW_Push, SW27 SW_Push, SW28 SW_Push, SW29 SW_Push, SW3 SW_Push, SW30 SW_Push, SW31 SW_Push, SW32 SW_Push, SW33 SW_Push, SW34 SW_Push, SW35 SW_Push, SW36 SW_Push, SW37 SW_Push, SW38 SW_Push, SW39 SW_Push, SW4 SW_Push, SW40 SW_Push, SW41 SW_Push, SW42 SW_Push, SW43 SW_Push, SW44 SW_Push, SW45 SW_Push, SW46 SW_Push, SW47 SW_Push, SW48 SW_Push, SW49 SW_Push, SW5 SW_Push, SW50 SW_Push, SW51 SW_Push, SW52 SW_Push, SW53 SW_Push, SW54 SW_Push, SW55 SW_Push, SW56 SW_Push, SW57 SW_Push, SW58 SW_Push, SW59 SW_Push, SW6 SW_Push, SW60 SW_Push, SW61 SW_Push, SW62 SW_Push, SW63 SW_Push, SW64 SW_Push, SW65 SW_Push, SW66 SW_Push, SW67 SW_Push, SW68 SW_Push, SW69 SW_Push, SW7 SW_Push, SW70 SW_Push, SW71 SW_Push, SW72 SW_Push, SW73 SW_Push, SW74 SW_Push, SW75 SW_Push, SW76 SW_Push, SW77 SW_Push, SW78 SW_Push, SW79 SW_Push, SW8 SW_Push, SW80 SW_Push, SW81 SW_Push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

Commit message: Add files via upload
Routing:
- net ROW3: track 853.1 -> 891.5 mm
- net ROW1: track 398.2 -> 412.8 mm
- added copper zone on B.Cu, net GND
Changed lines of the file:
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@@
 	)
 	(segment
-		(start 322 38)
-		(end 323.267 39.267)
-		(width 0.2)
-		(layer "B.Cu")
-		(net 1)
-	)
-	(segment
 		(start 152.7 47.5)
 		(end 162.26 47.5)
@@
 	)
 	(segment
+		(start 334.5 40.5)
+		(end 333 42)
+		(width 0.2)
+		(layer "B.Cu")
+		(net 1)
+	)
+	(segment
 		(start 257.475 47.5)
 		(end 267.035 47.5)
@@
 	)
 	(segment
-		(start 336.587 39.267)
-		(end 340.24 42.92)
+		(start 147.955 42.755)
+		(end 152.7 47.5)
 		(width 0.2)
 		(layer "B.Cu")
@@
 	)
 	(segment
-		(start 147.955 42.755)
-		(end 152.7 47.5)
+		(start 337.82 40.5)
+		(end 334.5 40.5)
 		(width 0.2)
 		(layer "B.Cu")
@@
 	)
 	(segment
+		(start 340.24 42.92)
+		(end 337.82 40.5)
+		(width 0.2)
+		(layer "B.Cu")
+		(net 1)
+	)
+	(segment
 		(start 293.245 42.755)
 		(end 300.375 35.625)
@@
 	)
 	(segment
+		(start 316.033 51.967)
+		(end 316 52)
+		(width 0.2)
+		(layer "B.Cu")
+		(net 1)
+	)
+	(segment
 		(start 90.7875 47.5)
 		(end 100.3475 47.5)
@@
 	)
 	(segment
+		(start 327.033 51.967)
+		(end 316.033 51.967)
+		(width 0.2)
+		(layer "B.Cu")
+		(net 1)
+	)
+	(segment
 		(start 43.18 42.755)
 		(end 47.925 47.5)
@@
 	)
 	(segment
-		(start 302.75 38)
-		(end 322 38)
-		(width 0.2)
-		(layer "B.Cu")
-		(net 1)
-	)
-	(segment
 		(start 286.085 47.5)
 		(end 290.83 42.755)
@@
 	)
 	(segment
+		(start 302.75 42.75)
+		(end 302.75 38)
+		(width 0.2)
+		(layer "B.Cu")
+		(net 1)
+	)
+	(segment
 		(start 209.8675 42.755)
 		(end 214.6125 47.5)
@@
 	)
 	(segment
+		(start 333 42)
+		(end 333 46)
+		(width 0.2)
+		(layer "B.Cu")
+		(net 1)
+	)
+	(segment
 		(start 66.9925 42.755)
 		(end 72.2065 47.969)
@@
 	)
 	(segment
+		(start 312 48)
+		(end 308 48)
+		(width 0.2)
+		(layer "B.Cu")
+		(net 1)
+	)
+	(segment
 		(start 371 35)
 		(end 348.16 35)
@@
 	)
 	(segment
+		(start 308 48)
+		(end 302.75 42.75)
+		(width 0.2)
+		(layer "B.Cu")
+		(net 1)
+	)
+	(segment
 		(start 300.375 35.625)
 		(end 302.75 38)
@@
 	)
 	(segment
-		(start 323.267 39.267)
-		(end 336.587 39.267)
+		(start 333 46)
+		(end 327.033 51.967)
+		(width 0.2)
+		(layer "B.Cu")
+		(net 1)
+	)
+	(segment
+		(start 316 52)
+		(end 312 48)
 		(width 0.2)
 		(layer "B.Cu")
@@
 	)
 	(segment
-		(start 162.385 95)
-		(end 167.005 90.38)
+		(start 32 94.5)
+		(end 43.8225 94.5)
 		(width 0.2)
 		(layer "B.Cu")
@@
 	)
 	(segment
-		(start 321.333 31.333)
-		(end 327.833 31.333)
+		(start 162.385 95)
+		(end 167.005 90.38)
 		(width 0.2)
 		(layer "B.Cu")
@@
 	)
 	(segment
-		(start 52.5625 95)
-		(end 67.135 95)
+		(start 377.5 78.5)
+		(end 377.5 153.5)
 		(width 0.2)
 		(layer "B.Cu")
@@
 	)
 	(segment
-		(start 373.373 33.873)
-		(end 376.5 37)
+		(start 52.5625 95)
+		(end 67.135 95)
 		(width 0.2)
 		(layer "B.Cu")
@@
 	)
 	(segment
-		(start 32 94.5)
-		(end 23.5 86)
-		(width 0.2)
-		(layer "B.Cu")
-		(net 17)
-	)
-	(segment
 		(start 268.669 96.794)
 		(end 274.891 96.794)
@@
 	)
 	(segment
+		(start 375 76)
+		(end 377.5 78.5)
+		(width 0.2)
+		(layer "B.Cu")
+		(net 17)
+	)
+	(segment
 		(start 200.485 95)
 		(end 205.105 90.38)
@@
 	)
 	(segment
-		(start 330.373 33.873)
-		(end 373.373 33.873)
+		(start 370 161)
+		(end 32.5 161)
 		(width 0.2)
 		(layer "B.Cu")
@@
 	)
 	(segment
-		(start 43.8225 94.5)
-		(end 32 94.5)
+		(start 24.5 153)
+		(end 24.5 102)
 		(width 0.2)
 		(layer "B.Cu")
@@
 	)
 	(segment
-		(start 27.5 30)
-		(end 320 30)
-		(width 0.2)
-		(layer "B.Cu")
-		(net 17)
-	)
-	(segment
 		(start 167.005 90.38)
 		(end 171.625 95)
@@
 	)
 	(segment
-		(start 205.105 90.38)
-		(end 209.725 95)
-		(width 0.2)
-		(layer "B.Cu")
-		(net 17)
-	)
-	(segment
-		(start 23.5 34)
-		(end 27.5 30)
+		(start 24.5 102)
+		(end 32 94.5)
 		(width 0.2)
 		(layer "B.Cu")
@@
 	)
 	(segment
-		(start 327.833 31.333)
-		(end 330.373 33.873)
+		(start 205.105 90.38)
+		(end 209.725 95)
 		(width 0.2)
 		(layer "B.Cu")
@@
 	)
 	(segment
-		(start 47.9425 90.38)
-		(end 43.8225 94.5)
-		(width 0.2)
-		(layer "B.Cu")
-		(net 17)
-	)
-	(segment
-		(start 376.5 74.5)
-		(end 375 76)
+		(start 377.5 153.5)
+		(end 370 161)
 		(width 0.2)
 		(layer "B.Cu")
@@
 	)
 	(segment
-		(start 376.5 37)
-		(end 376.5 74.5)
-		(width 0.2)
-		(layer "B.Cu")
-		(net 17)
-	)
-	(segment
-		(start 320 30)
-		(end 321.333 31.333)
+		(start 43.8225 94.5)
+		(end 47.9425 90.38)
 		(width 0.2)
 		(layer "B.Cu")
@@
 	)
 	(segment
-		(start 247.825 95)
-		(end 257.635 95)
+		(start 32.5 161)
+		(end 24.5 153)
 		(width 0.2)
 		(layer "B.Cu")
@@
 	)
 	(segment
-		(start 23.5 86)
-		(end 23.5 34)
+		(start 247.825 95)
+		(end 257.635 95)
 		(width 0.2)
 		(layer "B.Cu")
@@
 			)
 		)
+	)
+	(zone
+		(net 98)
+		(net_name "GND")
+		(layer "B.Cu")
+		(hatch edge 0.5)
+		(priority 1)
+		(connect_pads
+			(clearance 0.5)
+		)
+		(min_thickness 0.25)
+		(filled_areas_thickness no)
+		(fill yes
+			(thermal_gap 0.5)
+			(thermal_bridge_width 0.5)
+			(island_removal_mode 2)
+			(island_area_min 20)
+		)
+		(polygon
+			(pts
+				(xy 665.5 516) (xy 664 -112) (xy -160.5 -120.5) (xy -108 532)
+			)
+		)

Commit message: Add files via upload
Parts:
- moved MT1 1.27 mm to (304.8, 43.2)
Routing:
- net ROW5: track 494.7 -> 498.0 mm
- net ROW3: track 891.5 -> 890.0 mm
- net Net-(D85-A): track 4.05 -> 5.00 mm
- net COL14: track 259.2 -> 258.4 mm

Commit message: Add files via upload
Parts:
- added G***: LOGO, LOGO, F.Cu at (323.2, 107.2)
- added G***: LOGO, LOGO, F.Cu at (319.9, 126.3)
- added G***: LOGO, LOGO, B.Cu at (333.9, 107.2)
- SW44: footprint Button_Switch_Keyboard:SW_Cherry_MX_ISOEnter_PCB -> keyboardkey:SW_Cherry_MX_ISOEnter_PCB_v2
- moved D85 8.23 mm to (294.9, 36.1), turned to 90 degrees
- moved D10 4.76 mm to (233.7, 41.1)
- moved D7 4.76 mm to (171.8, 41.1)
- moved D3 4.76 mm to (90.8, 41.1)
- moved D4 4.76 mm to (109.9, 41.1)
- moved SW4 4.76 mm to (104.8, 38.1)
- moved SW2 4.76 mm to (66.7, 38.1)
- moved D2 4.76 mm to (71.8, 41.1)
- moved D6 4.76 mm to (152.7, 41.1)
- moved SW10 4.76 mm to (228.6, 38.1)
- moved SW3 4.76 mm to (85.7, 38.1)
- moved SW6 4.76 mm to (147.6, 38.1)
- moved SW7 4.76 mm to (166.7, 38.1)
- moved MT1 2.49 mm to (302.3, 43.2)
Connections:
- U1 pad 18: Net-(Brd1-SCL) -> Net-(Brd1-SDA)
- U1 pad 24: Net-(Brd1-SDA) -> Net-(Brd1-SCL)
Routing:
- net Net-(D44-A): track 11.9 -> 5.14 mm
- net ROW1: track 412.8 -> 407.9 mm
- net GPIO2: track 68.6 -> 72.3 mm
- net GPIO3: track 56.1 -> 59.8 mm
- net COL7: track 410.2 -> 407.4 mm
- net COL3: track 378.3 -> 375.5 mm
- net COL2: track 394.8 -> 392.0 mm
- net COL4: track 409.7 -> 406.9 mm
- net COL6: track 426.5 -> 423.7 mm
- net ROW6: track 787.3 -> 789.3 mm
- net COL10: track 229.3 -> 231.2 mm
- net COL14: track 258.4 -> 259.7 mm
- net Net-(Brd1-SCL): track 352.5 -> 351.7 mm
- net Net-(Brd1-SDA): track 38.5 -> 39.3 mm
- net Net-(D85-A): track 5.00 -> 5.61 mm
Other:
- board text added: "BAR"
- board text added: "DIY Keyboard"
- board text added: "Designed by Moritz Prenner"
- board text added: "OLED screen goes here!"
- board text added: "RP2040 pro micro"
- board text added: "SPACE"
- board text added: "Source here!"
