File: DIY_Keyboard.kicad_sch (KiCad schematic)
At the start: 170 parts, among them SW1 SW_Push, SW10 SW_Push, SW11 SW_Push, SW12 SW_Push, SW13 SW_Push, SW14 SW_Push, SW15 SW_Push, SW16 SW_Push, SW17 SW_Push, SW18 SW_Push, SW19 SW_Push, SW2 SW_Push, SW20 SW_Push, SW21 SW_Push, SW22 SW_Push, SW23 SW_Push, SW24 SW_Push, SW25 SW_Push, SW26 SW_Push, SW27 SW_Push, SW28 SW_Push, SW29 SW_Push, SW3 SW_Push, SW30 SW_Push, SW31 SW_Push, SW32 SW_Push, SW33 SW_Push, SW34 SW_Push, SW35 SW_Push, SW36 SW_Push, SW37 SW_Push, SW38 SW_Push, SW39 SW_Push, SW4 SW_Push, SW40 SW_Push, SW41 SW_Push, SW42 SW_Push, SW43 SW_Push, SW44 SW_Push, SW45 SW_Push, SW46 SW_Push, SW47 SW_Push, SW48 SW_Push, SW49 SW_Push, SW5 SW_Push, SW50 SW_Push, SW51 SW_Push, SW52 SW_Push, SW53 SW_Push, SW54 SW_Push, SW55 SW_Push, SW56 SW_Push, SW57 SW_Push, SW58 SW_Push, SW59 SW_Push, SW6 SW_Push, SW60 SW_Push, SW61 SW_Push, SW62 SW_Push, SW63 SW_Push, SW64 SW_Push, SW65 SW_Push, SW66 SW_Push, SW67 SW_Push, SW68 SW_Push, SW69 SW_Push, SW7 SW_Push, SW70 SW_Push, SW71 SW_Push, SW72 SW_Push, SW73 SW_Push, SW74 SW_Push, SW75 SW_Push, SW76 SW_Push, SW77 SW_Push, SW78 SW_Push, SW79 SW_Push, SW8 SW_Push, SW80 SW_Push, SW81 SW_Push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

Commit message: Add files via upload
Parts:
- SW44: footprint Button_Switch_Keyboard:SW_Cherry_MX_ISOEnter_PCB -> keyboardkey:SW_Cherry_MX_ISOEnter_PCB_v2
Connections:
- net at Brd1.3 (SCL): now also U1.24 (GP24); no longer U1.18 (GP18)
- net at Brd1.4 (SDA): now also U1.18 (GP18); no longer U1.24 (GP24)
Changed lines of the file:
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@@
 	(wire
 		(pts
-			(xy 373.38 181.61) (xy 374.65 181.61)
+			(xy 373.38 181.61) (xy 375.92 181.61)
 		)
 		(stroke
@@
 	(wire
 		(pts
+			(xy 374.65 182.88) (xy 370.84 182.88)
+		)
+		(stroke
+			(width 0)
+			(type default)
+		)
+	)
+	(wire
+		(pts
 			(xy 121.92 46.99) (xy 135.89 46.99)
 		)
@@
 	(wire
 		(pts
+			(xy 377.19 186.69) (xy 377.19 195.58)
+		)
+		(stroke
+			(width 0)
+			(type default)
+		)
+	)
+	(wire
+		(pts
 			(xy 297.18 46.99) (xy 307.34 46.99)
 		)
@@
 	(wire
 		(pts
-			(xy 370.84 182.88) (xy 377.19 182.88)
-		)
-		(stroke
-			(width 0)
-			(type default)
-		)
-	)
-	(wire
-		(pts
 			(xy 212.09 107.95) (xy 227.33 107.95)
 		)
@@
 	(wire
 		(pts
+			(xy 375.92 186.69) (xy 377.19 186.69)
+		)
+		(stroke
+			(width 0)
+			(type default)
+		)
+	)
+	(wire
+		(pts
 			(xy 149.86 66.04) (xy 165.1 66.04)
 		)
@@
 	(wire
 		(pts
+			(xy 375.92 181.61) (xy 375.92 186.69)
+		)
+		(stroke
+			(width 0)
+			(type default)
+		)
+	)
+	(wire
+		(pts
 			(xy 212.09 66.04) (xy 227.33 66.04)
 		)
@@
 	(wire
 		(pts
-			(xy 125.73 138.43) (xy 125.73 154.94)
+			(xy 374.65 195.58) (xy 374.65 182.88)
 		)
 		(stroke
@@
 	(wire
 		(pts
-			(xy 377.19 182.88) (xy 377.19 195.58)
+			(xy 125.73 138.43) (xy 125.73 154.94)
 		)
 		(stroke
@@
 	(wire
 		(pts
-			(xy 374.65 181.61) (xy 374.65 195.58)
-		)
-		(stroke
-			(width 0)
-			(type default)
-		)
-	)
-	(wire
-		(pts
 			(xy 135.89 146.05) (xy 149.86 146.05)
 		)
@@
 			)
 		)
-		(property "Footprint" "Button_Switch_Keyboard:SW_Cherry_MX_ISOEnter_PCB"
+		(property "Footprint" "keyboardkey:SW_Cherry_MX_ISOEnter_PCB_v2"
 			(at 236.22 73.66 0)
 			(effects
